File: v0/e90-dsi-split.kicad_pcb (KiCad board)
At the start: 2 copper layers, 33.9 x 22.1 mm, 12 parts, among them J1 3-2328724-1, J2 BM23PF0.8-40DP-0.35V_51_, J3 I2C Pinstack, J4 GPIO Pinstack

Commit message: next
Parts:
- added TP10: +5V5 Src, TestPoint:TestPoint_Pad_1.0x1.0mm, F.Cu at (100.8, 54.2)
- added TP11: VDD3V3_SYS, TestPoint:TestPoint_Pad_1.0x1.0mm, F.Cu at (106.5, 49.0)
- added TP11: +5V5 Screen, TestPoint:TestPoint_Pad_1.0x1.0mm, F.Cu at (100.8, 51.5)
- added TP11: VDD3V3_SYS, TestPoint:TestPoint_Pad_1.0x1.0mm, F.Cu at (109.0, 49.0)
- added TP9: GND Test, TestPoint:TestPoint_Pad_1.0x1.0mm, F.Cu at (98.4, 49.1)
- TP1: value +5V5 Test -> +5V5 Screen
- TP2: value -5V5 Test -> -5V5 Screen
- TP3: value AOI Test -> MVDD Test
- moved TP3 19.0 mm to (82.3, 49.1)
- moved TP5 15.6 mm to (79.9, 49.1)
- moved J4 9.34 mm to (88.5, 63.5)
- moved TP1 8.04 mm to (94.4, 54.2)
- moved TP2 7.68 mm to (94.4, 51.6)
- moved J3 6.22 mm to (93.1, 63.5)
- moved TP6 4.63 mm to (84.1, 63.4)
- moved TP8 1.54 mm to (84.8, 49.1)
- moved TP7 0.54 mm to (87.0, 49.1)
- moved TP4 0.21 mm to (89.2, 49.1)
Connections:
- J1 pad 14: /DATAP2 -> /CLK_P
- J1 pad 15: /DATAN2 -> /CLK_N
- J2 pad 39: -5V5_BL -> /AVEE
- J2 pad 40: +5V5_BL -> /AVDD
- J2 pad 5: /CLKN -> /CLK_N
- J2 pad 7: /CLKP -> /CLK_P
- TP1 pad 1: +5V5_BL -> /AVDD
- TP2 pad 1: -5V5_BL -> /AVEE
- TP3 pad 1: /EN_AOI -> /MVDD
Routing:
- net /DATAP2: track 34.2 -> 0.00 mm, vias 2 -> 0
- net /CLK_P: track 0.00 -> 29.7 mm
- net /DATAN2: track 27.9 -> 0.00 mm, vias 4 -> 0
- net /CLK_N: track 0.00 -> 26.4 mm, vias 0 -> 2
- net GND: track 55.0 -> 34.8 mm, vias 5 -> 0
- net /AVEE: track 0.00 -> 20.0 mm, vias 0 -> 2
- net +5V5_BL: track 28.8 -> 10.9 mm
- net /AVDD: track 0.00 -> 17.9 mm, vias 0 -> 2
- net -5V5_BL: track 27.6 -> 13.3 mm
- net /IM_0: track 26.3 -> 14.5 mm, vias 4 -> 1
- net /ELVDD: track 4.48 -> 15.7 mm, vias 0 -> 2
- net /RL_SEL: track 23.5 -> 13.8 mm, vias 0 -> 1
- net /MVDD: track 0.00 -> 6.28 mm
- net /SCL: track 19.2 -> 13.1 mm, vias 0 -> 1
- net /VGMP: track 10.6 -> 6.37 mm
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Other:
- board size 33.9 x 22.1 mm -> 33.5 x 17.6 mm
- rule pad_to_mask_clearance: 0 -> 0.0508
- board text added: "EL"
- board text added: "GND"
- board text added: "MIPI Mapper [v1] TJM 2025"
- board text added: "MP"
- board text added: "MV"
- board text added: "SP"
- board text added: "V1"
- board text removed: "AOI"
- board text removed: "ELVDD"
- board text removed: "MIPI Mapper [v0] TJM 2025"
- board text removed: "VGMP"
- board text removed: "VGSP"
- board text removed: "VREF1"

Commit message: misc updates, move to v1
Parts:
- J1: footprint Library:CONN-SMD_FH26W-31S-0.3SHW-60 -> bacon:FPC-SMD_31P-P0.30_HDGC_0.3K-QX-31PWB
- J2: footprint Library:CONN-SMD_BM23PF0.8-40DS-0.35V880 -> bacon:BM23PF0840DS035V51-GOOD

Commit message: v1
Parts:
- removed J3: I2C Pinstack, Connector_PinHeader_1.00mm:PinHeader_1x03_P1.00mm_Horizontal
- removed J4: GPIO Pinstack, Connector_PinHeader_1.00mm:PinHeader_1x03_P1.00mm_Horizontal
- removed the TP11 at (106.5, 49.0)
- removed the TP11 at (100.8, 51.5)
- removed the TP11 at (109.0, 49.0)
- removed TP6: GPIO Test, TestPoint:TestPoint_Pad_1.0x1.0mm
- added C1: 47 uF, Capacitor_SMD:C_1206_3216Metric, B.Cu at (102.0, 80.2)
- added FPC1: F0504-H-06-10G-R, bacon:FFC-SMD_6P-P0.50_F0504-H-06-10G-R, F.Cu at (112.8, 80.8)
- added REF**: PinHeader_1x14_P2.54mm_Vertical, Connector_PinHeader_2.54mm:PinHeader_1x14_P2.54mm_Vertical, F.Cu at (81.5, 96.5)
- added REF**: PinHeader_1x14_P2.54mm_Vertical, Connector_PinHeader_2.54mm:PinHeader_1x14_P2.54mm_Vertical, F.Cu at (81.5, 76.0)
- added TP11: -5V5 Screen, TestPoint:TestPoint_Pad_1.0x1.0mm, B.Cu at (98.0, 80.0)
- added U1: ICM-42605, footprints:LGA14_2P5X3X0P91_IVS, F.Cu at (107.0, 80.1)
- added U2: LM2665M6, Package_TO_SOT_SMD:SOT-23-6, F.Cu at (101.9, 80.5)
- TP1, TP10, TP2, TP3, TP4, TP5, TP7, TP8, TP9: moved to B.Cu
- moved TP5 44.0 mm to (82.0, 93.0), turned to 180 degrees
- moved TP3 43.9 mm to (84.2, 93.0), turned to 180 degrees
- moved TP9 36.4 mm to (108.8, 84.0), turned to 180 degrees
- moved TP4 33.5 mm to (81.8, 81.8), turned to 180 degrees
- moved J1 32.7 mm to (112.8, 89.2), turned to -90 degrees
- moved TP7 30.6 mm to (81.8, 79.2), turned to 180 degrees
- moved J2 30.4 mm to (88.2, 87.1), turned to 0 degrees
- moved TP8 30.2 mm to (84.2, 79.2), turned to 180 degrees
- moved TP2 28.4 mm to (95.2, 80.0), turned to 180 degrees
- moved TP10 28.2 mm to (98.0, 82.2), turned to 180 degrees
- moved TP1 28.1 mm to (95.2, 82.2), turned to 180 degrees
Connections:
- net +5V5_BL renamed LCD0_BL+
- net -5V5_BL renamed LCD0_BL-
- J1 pad 32: unconnected-(J1-Pad32) -> GND
- J1 pad 33: unconnected-(J1-Pad33) -> GND
- J2 pad 28: /SDA -> unconnected-(J2-Pad28)
- J2 pad 30: /SCL -> unconnected-(J2-Pad30)
- J2 pad 37: GND -> /OTP_PWR
- J2 pad 38: /AVSS -> GND
- J2 pad MP1: (no net) -> VDD1V8_SYS
- J2 pad MP2: (no net) -> VDD1V8_SYS
- J2 pad MP3: (no net) -> VDD1V8_SYS
- J2 pad MP4: (no net) -> VDD1V8_SYS
Routing:
- net VDD1V8_SYS: track 6.10 -> 58.5 mm, vias 0 -> 2
- net /EN_AOI: track 20.4 -> 0.00 mm
- net /IM_0: track 14.5 -> 0.00 mm, vias 1 -> 0
- net /SDA: track 22.8 -> 8.70 mm, vias 4 -> 0
- net /RL_SEL: track 13.8 -> 0.00 mm, vias 1 -> 0
- net LCD0_BL+: track 10.9 -> 24.1 mm, vias 2 -> 4
- net /AVDD: track 17.9 -> 5.63 mm, vias 2 -> 1
- net /INT: track 0.00 -> 11.0 mm, vias 0 -> 2
- net /AVEE: track 20.0 -> 9.80 mm, vias 2 -> 1
- net /ELVDD: track 15.7 -> 6.18 mm, vias 2 -> 1
- net /GPIO: track 8.89 -> 0.00 mm
- net /DATAP1: track 26.5 -> 34.2 mm, vias 2 -> 0
- net GND: track 34.8 -> 42.5 mm, vias 0 -> 2
- net VDD3V3_SYS: track 3.94 -> 11.6 mm, vias 0 -> 2
- net LCD0_BL-: track 13.3 -> 20.9 mm, vias 2 -> 4
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Other:
- board size 33.5 x 17.6 mm -> 35.6 x 22.9 mm
- board text removed: "+5V5"
- board text removed: "-5V5"
- board text removed: "CFG"
- board text removed: "EL"
- board text removed: "GND"
- board text removed: "GPIO"
- board text removed: "I2C"
- board text removed: "MP"
- board text removed: "MV"
- board text removed: "SP"
- board text removed: "V1"

Commit message: v1 updates
Parts:
- moved J1 30.2 mm to (113.3, 59.1)
- moved C1 24.1 mm to (102.0, 56.1)
- moved J2 24.1 mm to (88.2, 62.9)
- moved REF** 24.1 mm to (81.5, 72.4)
- moved REF** 24.1 mm to (81.5, 51.9)
- moved TP1 24.1 mm to (95.2, 58.1)
- moved TP10 24.1 mm to (98.0, 58.1)
- moved TP11 24.1 mm to (98.0, 55.9)
- moved TP2 24.1 mm to (95.2, 55.9)
- moved TP3 24.1 mm to (84.2, 68.9)
- moved TP4 24.1 mm to (81.8, 57.6)
- moved TP5 24.1 mm to (82.0, 68.9)
- moved TP7 24.1 mm to (81.8, 55.1)
- moved TP8 24.1 mm to (84.2, 55.1)
- moved U2 24.1 mm to (101.9, 56.3)
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Connections:
- FPC1 pad 1: /SDA -> GND
- FPC1 pad 2: /SCL -> VDD3V3_SYS
- FPC1 pad 3: /RST -> /INT
- FPC1 pad 4: /INT -> /RST
- FPC1 pad 5: VDD3V3_SYS -> /SCL
- FPC1 pad 6: GND -> /SDA
- J1 pad 1: LCD0_BL+ -> VDD3V3_SYS
- J1 pad 11: unconnected-(J1-Pad11) -> /DATAN0
- J1 pad 12: unconnected-(J1-Pad12) -> /DATAP0
- J1 pad 14: /CLK_P -> /DATAN1
- J1 pad 15: /CLK_N -> /DATAP1
- J1 pad 17: /DATAP1 -> /CLK_N
- J1 pad 18: /DATAN1 -> /CLK_P
- J1 pad 2: LCD0_BL+ -> VDD3V3_SYS
- J1 pad 20: /DATAP0 -> unconnected-(J1-Pad20)
- J1 pad 21: /DATAN0 -> unconnected-(J1-Pad21)
- J1 pad 23: unconnected-(J1-Pad23) -> GND
- J1 pad 24: unconnected-(J1-Pad24) -> LCD0_BL-
- J1 pad 25: GND -> LCD0_BL-
- J1 pad 26: VDD1V8_SYS -> LCD0_BL-
- J1 pad 27: /RESET -> LCD0_BL-
- J1 pad 28: GND -> unconnected-(J1-Pad28)
- J1 pad 29: VDD1V8_SYS -> LCD0_BL+
- J1 pad 3: LCD0_BL+ -> VDD1V8_SYS
- J1 pad 30: VDD3V3_SYS -> LCD0_BL+
- J1 pad 31: VDD3V3_SYS -> LCD0_BL+
- J1 pad 4: unconnected-(J1-Pad4) -> GND
- J1 pad 5: LCD0_BL- -> /RESET
- J1 pad 6: LCD0_BL- -> VDD1V8_SYS
- J1 pad 7: LCD0_BL- -> GND
- J1 pad 8: LCD0_BL- -> unconnected-(J1-Pad8)
- J1 pad 9: GND -> unconnected-(J1-Pad9)
- J2 pad 28: unconnected-(J2-Pad28) -> /SDA_D
- J2 pad 30: unconnected-(J2-Pad30) -> /SCL_D
Routing:
- net VDD1V8_SYS: track 58.5 -> 39.6 mm, vias 2 -> 4
- net /CLK_P: track 30.9 -> 40.1 mm
- net /CLK_N: track 33.9 -> 40.2 mm, vias 0 -> 2
- net /DATAP0: track 31.2 -> 36.7 mm
- net /DATAN0: track 31.1 -> 36.6 mm
- net /SCL: track 8.00 -> 12.4 mm, vias 0 -> 2
- net /SDA: track 8.70 -> 13.0 mm
- net /INT: track 11.0 -> 8.13 mm, vias 2 -> 0
- net LCD0_BL+: track 24.1 -> 21.2 mm, vias 4 -> 2
- net LCD0_BL-: track 20.9 -> 19.2 mm, vias 4 -> 2
- net VDD3V3_SYS: track 11.6 -> 13.2 mm
- net GND: track 42.5 -> 41.1 mm, vias 2 -> 1
- net /RESET: track 28.0 -> 28.9 mm
- added copper zone on B.Cu, net (none)
- added copper zone on F.Cu, net (none)
- added copper zone on F.Cu, net GND

Commit message: v1 updates
Parts:
- removed U2: LM2665M6, Package_TO_SOT_SMD:SOT-23-6
- added C2: 1uF, Capacitor_SMD:C_0603_1608Metric, B.Cu at (103.8, 56.8)
- added D1: ~, Diode_SMD:D_SOD-123, F.Cu at (100.0, 58.2)
- added L1: 220uH, Inductor_SMD:L_TDK_NLV32_3.2x2.5mm, B.Cu at (109.2, 56.2)
- added R1: 65k, Resistor_SMD:R_0603_1608Metric, F.Cu at (105.5, 55.5)
- added R2: 10k, Resistor_SMD:R_0603_1608Metric, F.Cu at (107.0, 55.5)
- added U3: LTC3638xMSE, Package_SO:Analog_MSOP-12-16-1EP_3x4.039mm_P0.5mm_EP1.651x2.845mm, B.Cu at (100.1, 56.5)
- C1: value 47 uF -> 10uF; footprint Capacitor_SMD:C_1206_3216Metric -> Capacitor_SMD:C_1210_3225Metric
- moved C1 8.50 mm to (93.5, 56.2), turned to 90 degrees
- moved TP10 8.32 mm to (89.8, 57.0)
- moved TP11 8.29 mm to (89.8, 55.0)
- moved TP1 7.83 mm to (87.5, 57.0)
- moved TP2 7.80 mm to (87.5, 55.0)
Connections:
- C1 pad 1: Net-(U2-CAP+) -> LCD0_BL-
- C1 pad 2: Net-(U2-CAP-) -> -5V5
Routing:
- net -5V5: track 2.98 -> 25.6 mm, vias 1 -> 2
- net LCD0_BL-: track 19.2 -> 36.2 mm, vias 2 -> 3
- net LCD0_BL+: track 21.2 -> 31.0 mm, vias 2 -> 1
- net Net-(U3-SW): track 0.00 -> 7.08 mm
- net Net-(D1-K): track 0.00 -> 6.98 mm
- net /DATAN0: track 36.6 -> 30.7 mm
- net Net-(U2-CAP+): track 3.67 -> 0.00 mm, vias 1 -> 0
- net Net-(U2-CAP-): track 3.37 -> 0.00 mm, vias 1 -> 0
- net VDD1V8_SYS: track 39.6 -> 42.1 mm
- net /AVDD: track 5.63 -> 7.14 mm
- net /AVEE: track 9.80 -> 11.1 mm
- net /RESET: track 28.9 -> 28.3 mm

Commit message: v1 updates
Connections:
- net -5V5 renamed -6V
Routing:
- net LCD0_BL+: track 31.0 -> 43.0 mm, vias 1 -> 3
- net /DATAN0: track 30.7 -> 36.6 mm
- net Net-(U3-SS): track 0.00 -> 4.71 mm
- net Net-(D1-K): track 6.98 -> 11.3 mm, vias 0 -> 1
- net -6V: track 25.6 -> 27.4 mm

Commit message: v1: hopefully final
Parts:
- C2: renamed from C1; value 10uF -> 100uF; footprint Capacitor_SMD:C_1210_3225Metric -> Capacitor_SMD:C_1206_3216Metric
- D1: footprint Diode_SMD:D_SOD-123 -> Diode_SMD:D_SOD-523
- L1: value 220uH -> 56uH; footprint Inductor_SMD:L_TDK_NLV32_3.2x2.5mm -> Inductor_SMD:L_1812_4532Metric
- moved TP4 1.15 mm to (81.8, 58.8)
- moved D1 0.35 mm to (99.8, 58.0)
- renumbered C2 to C1
Connections:
- U3 pad 10: Net-(U3-SS) -> unconnected-(U3-SS-Pad10)
- U3 pad 7: Net-(U3-SS) -> -6V
Routing:
- net Net-(U3-SS): track 4.71 -> 0.00 mm
- net Net-(D1-K): track 11.3 -> 12.4 mm
- net LCD0_BL-: track 35.7 -> 34.8 mm
- removed copper zone on B.Cu, net (none)
- removed copper zone on F.Cu, net (none)
- removed copper zone on F.Cu, net GND
Other:
- board text added: "+5v5"
- board text added: "-6v"
- board text added: "EL/MVDD"
- board text added: "Gamma"
- board text added: "VREF"

Commit message: updates post rework
Connections:
- L1 pad 1: Net-(U3-SW) -> Net-(D1-K)
- R1 pad 2: Net-(D1-K) -> Net-(U3-VFB)
- R2 pad 1: Net-(D1-K) -> Net-(U3-VFB)
- U3 pad 1: Net-(U3-SW) -> Net-(D1-K)
- U3 pad 9: Net-(D1-K) -> Net-(U3-VFB)
Routing:
- net Net-(U3-VFB): track 0.00 -> 11.3 mm, vias 0 -> 1
- net Net-(U3-SW): track 7.44 -> 0.00 mm
Changed lines of the file:
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@@
 			(psa4output no)
 			(plot_black_and_white yes)
-			(plotinvisibletext no)
 			(sketchpadsonfab no)
 			(plotpadnumbers no)
@@
 	(net 53 "-6V")
 	(net 54 "Net-(D1-K)")
-	(net 55 "Net-(U3-SW)")
+	(net 55 "Net-(U3-VFB)")
 	(net 56 "unconnected-(U3-FBO-Pad5)")
 	(net 57 "unconnected-(U3-ISET-Pad11)")
@@
 			(layers "F.Cu" "F.Mask" "F.Paste")
 			(roundrect_rratio 0.25)
-			(net 54 "Net-(D1-K)")
+			(net 55 "Net-(U3-VFB)")
 			(pintype "passive")
 		)
@@
 			(layers "F.Cu" "F.Mask" "F.Paste")
 			(roundrect_rratio 0.25)
-			(net 54 "Net-(D1-K)")
+			(net 55 "Net-(U3-VFB)")
 			(pintype "passive")
 		)
@@
 			(layers "B.Cu" "B.Mask" "B.Paste")
 			(roundrect_rratio 0.222222)
-			(net 55 "Net-(U3-SW)")
+			(net 54 "Net-(D1-K)")
 			(pintype "passive")
 		)
@@
 			(layers "B.Cu" "B.Mask" "B.Paste")
 			(roundrect_rratio 0.25)
-			(net 55 "Net-(U3-SW)")
+			(net 54 "Net-(D1-K)")
 			(pinfunction "SW")
 			(pintype "passive")
@@
 			(layers "B.Cu" "B.Mask" "B.Paste")
 			(roundrect_rratio 0.25)
-			(net 54 "Net-(D1-K)")
+			(net 55 "Net-(U3-VFB)")
 			(pinfunction "VFB")
 			(pintype "input")
@@
 	)
 	(segment
-		(start 100.9 59)
-		(end 101.65 58.25)
-		(width 0.1016)
+		(start 100.45 58)
+		(end 100.749999 58)
+		(width 0.2)
 		(layer "F.Cu")
 		(net 54)
 	)
 	(segment
-		(start 100 59)
-		(end 100.9 59)
-		(width 0.1016)
+		(start 100.749999 58)
+		(end 104 54.75)
+		(width 0.2)
 		(layer "F.Cu")
 		(net 54)
 	)
+	(via
+		(at 104 54.75)
+		(size 0.6)
+		(drill 0.3)
+		(layers "F.Cu" "B.Cu")
+		(net 54)
+	)
 	(segment
-		(start 101.925 58.25)
-		(end 105.5 54.675)
+		(start 102.311 54.65)
+		(end 102.211 54.75)
 		(width 0.1016)
-		(layer "F.Cu")
+		(layer "B.Cu")
 		(net 54)
 	)
 	(segment
-		(start 107 54.675)
-		(end 105.5 54.675)
+		(start 104 54.75)
+		(end 105 54.75)
 		(width 0.1016)
-		(layer "F.Cu")
+		(layer "B.Cu")
 		(net 54)
 	)
 	(segment
-		(start 100.45 58)
-		(end 100.45 58.55)
-		(width 0.2)
-		(layer "F.Cu")
+		(start 102.211 54.75)
+		(end 104 54.75)
+		(width 0.1016)
+		(layer "B.Cu")
 		(net 54)
 	)
 	(segment
-		(start 105.5 54.675)
-		(end 105.5 54.825)
+		(start 105 54.75)
+		(end 105.6375 54.1125)
 		(width 0.1016)
-		(layer "F.Cu")
+		(layer "B.Cu")
 		(net 54)
 	)
 	(segment
-		(start 101.65 58.25)
-		(end 101.925 58.25)
+		(start 105.6375 54.1125)
+		(end 109.25 54.1125)
 		(width 0.1016)
-		(layer "F.Cu")
+		(layer "B.Cu")
 		(net 54)
 	)
 	(segment
-		(start 100.45 58.55)
-		(end 100 59)
-		(width 0.2)
+		(start 100.9 59)
+		(end 101.65 58.25)
+		(width 0.1016)
 		(layer "F.Cu")
-		(net 54)
+		(net 55)
 	)
-	(via
-		(at 100 59)
-		(size 0.6)
-		(drill 0.3)
-		(layers "F.Cu" "B.Cu")
-		(net 54)
+	(segment
+		(start 100 59)
+		(end 100.9 59)
+		(width 0.1016)
+		(layer "F.Cu")
+		(net 55)
 	)
 	(segment
-		(start 98.75 59)
-		(end 100 59)
+		(start 101.925 58.25)
+		(end 105.5 54.675)
 		(width 0.1016)
-		(layer "B.Cu")
-		(net 54)
+		(layer "F.Cu")
+		(net 55)
 	)
 	(segment
-		(start 98 58.25)
-		(end 98.75 59)
+		(start 107 54.675)
+		(end 105.5 54.675)
 		(width 0.1016)
-		(layer "B.Cu")
-		(net 54)
+		(layer "F.Cu")
+		(net 55)
 	)
 	(segment
-		(start 102.311 54.65)
-		(end 102.211 54.75)
+		(start 105.5 54.675)
+		(end 105.5 54.825)
 		(width 0.1016)
-		(layer "B.Cu")
+		(layer "F.Cu")
 		(net 55)
 	)
 	(segment
-		(start 102.211 54.75)
-		(end 105 54.75)
+		(start 101.65 58.25)
+		(end 101.925 58.25)
 		(width 0.1016)
-		(layer "B.Cu")
+		(layer "F.Cu")
+		(net 55)
+	)
+	(via
+		(at 100 59)
+		(size 0.6)
+		(drill 0.3)
+		(layers "F.Cu" "B.Cu")
 		(net 55)
 	)
 	(segment
-		(start 105 54.75)
-		(end 105.6375 54.1125)
+		(start 98.75 59)
+		(end 100 59)
 		(width 0.1016)
 		(layer "B.Cu")
@@
 	)
 	(segment
-		(start 105.6375 54.1125)
-		(end 109.25 54.1125)
+		(start 98 58.25)
+		(end 98.75 59)
 		(width 0.1016)
 		(layer "B.Cu")
