File: v0/e90-dsi-split.kicad_pcb (KiCad board)
At the start: 2 copper layers, 35.6 x 22.9 mm, 30 parts, among them J1 3-2328724-1, J2 BM23PF0.8-40DP-0.35V_51_, U1 ICM-42605, U3 LTC3638xMSE

Commit message: v2: more updates
Parts:
- added C14: C_Small, Capacitor_SMD:C_0603_1608Metric, B.Cu at (89.0, 66.3)
- moved C11 4.02 mm to (96.2, 61.4)
- moved D2 1.43 mm to (96.6, 63.3)
Connections:
- J1 pad 29: unconnected-(J1-Pad29) -> LCD0_BL+
- J1 pad 30: unconnected-(J1-Pad30) -> LCD0_BL+
- J1 pad 31: unconnected-(J1-Pad31) -> LCD0_BL+
- J2 pad 27: /IM_0 -> GND
- J2 pad 38: unconnected-(J2-Pad38) -> GND
- TP10 pad 1: VDD3V3_SYS -> LCD0_BL+
Routing:
- net LCD0_BL+: track 0.00 -> 22.5 mm, vias 0 -> 2
- net VDD3V3_SYS: track 22.2 -> 0.00 mm, vias 2 -> 0
- net GND: track 120.2 -> 109.0 mm
- net /VDD: track 10.7 -> 5.37 mm
- net /MVDD: track 0.00 -> 2.90 mm, vias 0 -> 1
- net /VREF1: track 12.3 -> 11.6 mm
- net /VCOM: track 23.3 -> 22.7 mm
- removed copper zone on B.Cu, net GND
Other:
- board size 35.6 x 22.9 mm -> 36.2 x 22.9 mm
