File: v0/e90-dsi-split.kicad_sch (KiCad schematic)
At the start: 12 parts, among them J1 3-2328724-1, J2 BM23PF0.8-40DP-0.35V_51_, J3 I2C Pinstack, J4 GPIO Pinstack

Commit message: next
Parts:
- added TP10: +5V5 Src, TestPoint:TestPoint_Pad_1.0x1.0mm, symbol Connector:TestPoint
- added TP11: +5V5 Screen, TestPoint:TestPoint_Pad_1.0x1.0mm, symbol Connector:TestPoint
- added TP9: GND Test, TestPoint:TestPoint_Pad_1.0x1.0mm, symbol Connector:TestPoint
- TP1: value +5V5 Test -> +5V5 Screen
- TP2: value -5V5 Test -> -5V5 Screen
- TP3: value AOI Test -> MVDD Test
Connections:
- net +5V5_BL: now also TP10.1; no longer J2.40, TP1.1
- net -5V5_BL: now also TP11.1; no longer J2.39, TP2.1
- net DATAN2: no longer J1.15
- net DATAP2: no longer J1.14
- net EN_AOI: no longer TP3.1
- net GND: now also TP9.1
- net MVDD: now also TP3.1
- net CLKN renamed CLK_N
- net CLK_N: now also J1.15
- net CLKP renamed CLK_P
- net CLK_P: now also J1.14
- new net AVDD: J2.40, TP1.1
- new net AVEE: J2.39, TP2.1
- no-connect marks 11 -> 9
Other:
- note added: "NOTE: Pads to be bridged before use"

Commit message: misc updates, move to v1
Parts:
- J1: footprint Library:CONN-SMD_FH26W-31S-0.3SHW-60 -> bacon:FPC-SMD_31P-P0.30_HDGC_0.3K-QX-31PWB; symbol 3-2328724-1:3-2328724-1 -> bacon:0.3K-QX-31PWB; Manufacturer (none) -> HDGC(华德共创); Manufacturer Part (none) -> 0.3K-QX-31PWB; Supplier (none) -> LCSC; Supplier Part (none) -> C2919512
- J2: footprint Library:CONN-SMD_BM23PF0.8-40DS-0.35V880 -> bacon:HRS_BM23PF0.8-40DS-0.35V_51_; symbol BM23PF0.8-40DP-0.35V_51_:BM23PF0.8-40DP-0.35V_51_ -> BM23PF0.8-40DS-0.35V_51_:BM23PF0.8-40DS-0.35V_51_
Connections:
- net GND: no longer J1.S1 (SHIELD), J1.S2 (SHIELD)

Commit message: v1
Parts:
- removed J3: I2C Pinstack, Connector_PinHeader_1.00mm:PinHeader_1x03_P1.00mm_Horizontal, symbol Connector_Generic_MountingPin:Conn_01x03_MountingPin
- removed J4: GPIO Pinstack, Connector_PinHeader_1.00mm:PinHeader_1x03_P1.00mm_Horizontal, symbol Connector_Generic_MountingPin:Conn_01x03_MountingPin
- removed TP6: GPIO Test, TestPoint:TestPoint_Pad_1.0x1.0mm, symbol Connector:TestPoint
- added C1: 47 uF, Capacitor_SMD:C_1206_3216Metric, symbol Device:C_Polarized_Small
- added FPC1: F0504-H-06-10G-R, bacon:FFC-SMD_6P-P0.50_F0504-H-06-10G-R, symbol bacon:F0504-H-06-10G-R
- added U1: ICM-42605, footprints:LGA14_2P5X3X0P91_IVS, symbol 2025-04-06_22-45-15:ICM-42605
- added U2: LM2665M6, Package_TO_SOT_SMD:SOT-23-6, symbol Regulator_SwitchedCapacitor:LM2665M6
- J2: footprint bacon:HRS_BM23PF0.8-40DS-0.35V_51_ -> bacon:BM23PF0840DS035V51-GOOD
- TP11: value +5V5 Screen -> -5V5 Screen
Connections:
- net AVSS is gone; now on net GND: J2.38
- net GND: now also J1.32, J1.33, FPC1.6, FPC1.7, FPC1.8, U1.6 (GND); no longer J2.37
- net SCL: now also FPC1.2, U1.13 (AP_SCL/AP_SCLK); no longer J2.30
- net SDA: now also FPC1.1, U1.14 (AP_SDA/AP_SDIO/AP_SDI); no longer J2.28
- net VDD1V8_SYS: now also J2.MP1, J2.MP2, J2.MP3, J2.MP4; no longer J2.P1_1 (P1)
- net VDD3V3_SYS: now also FPC1.5, U1.5 (VDDIO), U1.8 (VDD)
- net +5V5_BL renamed LCD0_BL+
- net LCD0_BL+: now also U2.1 (V+)
- net -5V5_BL renamed LCD0_BL-
- net LCD0_BL-: now also U2.2 (GND), U2.4 (SD); no longer TP11.1
- removed net VDD: J2.P2_1 (P2)
- new net: C1.2, U2.3 (CAP-)
- new net: C1.1, U2.6 (CAP+)
- new net -5V5: TP11.1, U2.5 (OUT)
- new net INT: FPC1.4, U1.4 (INT1/INT)
- new net OTP_PWR: J2.37
- new net RST: FPC1.3
- no-connect marks 9 -> 18
Other:
- note added: "Board Display Interface"
- note added: "Board I2C Interface"
- note added: "IMU: ICM-42605"
- note added: "Microdisplay Interface"
- note added: "NOTES: - Not using fsync feature - I2C bus"
- note added: "NOTES: - Using LCD backlight driver for OLED 5v5 rail - Only 2 DSI lanes wired (really 3 but one is clk) - Clk lane mapping is arbitrary - Pins reverse direction of expected"
- note added: "Power System"
- note added: "Test Points"
- note removed: "NOTE: We will be abusing LCD0_BL to drive the 5.5V rail for the OLED."
- note removed: "NOTE: shared GND shouldn't matter? I think?"
- moved on the sheet: J2, TP1, TP10, TP11, TP2, TP3, TP4, TP5, TP7, TP8, TP9

Commit message: v1 updates
Connections:
- net CLK_N: now also J1.17; no longer J1.15
- net CLK_P: now also J1.18; no longer J1.14
- net DATAN0: now also J1.11; no longer J1.21
- net DATAN1: now also J1.14; no longer J1.18
- net DATAP0: now also J1.12; no longer J1.20
- net DATAP1: now also J1.15; no longer J1.17
- net GND: now also FPC1.1, J1.23, J1.4, J1.7; no longer FPC1.6, J1.25, J1.28, J1.9
- net INT: now also FPC1.3; no longer FPC1.4
- net LCD0_BL+: now also J1.29, J1.30, J1.31; no longer J1.1, J1.2, J1.3
- net LCD0_BL-: now also J1.24, J1.25, J1.26, J1.27; no longer J1.5, J1.6, J1.7, J1.8
- net RESET: now also J1.5; no longer J1.27
- net RST: now also FPC1.4; no longer FPC1.3
- net SCL: now also FPC1.5; no longer FPC1.2
- net SDA: now also FPC1.6; no longer FPC1.1
- net VDD1V8_SYS: now also J1.3, J1.6; no longer J1.26, J1.29
- net VDD3V3_SYS: now also FPC1.2, J1.1, J1.2; no longer FPC1.5, J1.30, J1.31
- net SDA_D: now reaches J2.28
- net SCL_D: now reaches J2.30
Other:
- note added: "NOTES: - Produce -5v5 for OLED cell - Cap for stabilization - Can be disabled by just not soldering 5v5 pads"
- moved on the sheet: C1, FPC1, TP1, TP10, TP11, TP2, TP3, TP4, TP5, TP7, TP8, TP9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

Commit message: v1 updates
Parts:
- removed C1: 47 uF, Capacitor_SMD:C_1206_3216Metric, symbol Device:C_Polarized_Small
- removed U2: LM2665M6, Package_TO_SOT_SMD:SOT-23-6, symbol Regulator_SwitchedCapacitor:LM2665M6
- added C1: 10uF, Capacitor_SMD:C_1210_3225Metric, symbol Device:C_Small
- added C2: 1uF, Capacitor_SMD:C_0603_1608Metric, symbol Device:C_Small
- added D1: ~, Diode_SMD:D_SOD-123, symbol Device:D_Zener_Small
- added L1: 220uH, Inductor_SMD:L_TDK_NLV32_3.2x2.5mm, symbol Device:L_Small
- added R1: 65k, Resistor_SMD:R_0603_1608Metric, symbol Device:R_Small_US
- added R2: 10k, Resistor_SMD:R_0603_1608Metric, symbol Device:R_Small_US
- added U3: LTC3638xMSE, Package_SO:Analog_MSOP-12-16-1EP_3x4.039mm_P0.5mm_EP1.651x2.845mm, symbol Regulator_Switching:LTC3638xMSE
Connections:
- net -5V5: now also C1.2, D1.2 (A), R2.2, U3.12 (OVLO), U3.16 (GND), U3.17 (GND), U3.6 (VPRG2), U3.8 (GND)
- net LCD0_BL+: now also C2.1, U3.14 (RUN), U3.3 (VIN)
- net LCD0_BL-: now also C1.1, C2.2, L1.2, R1.1
- new net: D1.1 (K), R1.2, R2.1, U3.9 (VFB)
- new net: L1.1, U3.1 (SW)
- new net: U3.10 (SS), U3.7 (VPRG1)
- no-connect marks 18 -> 19
Other:
- note added: "NOTES: - Produce -6V for OLED cell - Circuit based on Fig. 15 in LTC3638 DS"
- note removed: "NOTES: - Produce -5v5 for OLED cell - Cap for stabilization - Can be disabled by just not soldering 5v5 pads"

Commit message: v1 updates
Connections:
- net -5V5 renamed -6V
- no-connect marks 19 -> 20
Changed lines of the file:
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@@
 	)
 	(no_connect
+		(at 76.2 186.69)
+	)
+	(no_connect
 		(at 66.04 71.12)
 	)
@@
 			)
 		)
-		(property "Value" "-5V5"
-			(at 133.35 86.36 0)
+		(property "Value" "-6V"
+			(at 135.89 82.5499 0)
 			(effects
 				(font
 					(size 1.27 1.27)
 				)
+				(justify right)
 			)
 		)
@@
 			)
 		)
-		(property "Value" "-5V5"
+		(property "Value" "-6V"
 			(at 125.73 193.0399 90)
 			(effects

Commit message: v1: hopefully final
Parts:
- C2: renamed from C1; value 10uF -> 100uF; footprint Capacitor_SMD:C_1210_3225Metric -> Capacitor_SMD:C_1206_3216Metric
- D1: footprint Diode_SMD:D_SOD-123 -> Diode_SMD:D_SOD-523
- L1: value 220uH -> 56uH; footprint Inductor_SMD:L_TDK_NLV32_3.2x2.5mm -> Inductor_SMD:L_1812_4532Metric
- renumbered C2 to C1
Connections:
- net -6V: now also U3.7 (VPRG1)
- net at U3.10 (SS): no longer U3.7 (VPRG1)
- no-connect marks 20 -> 21
Other:
- note added: "C1: CL10B105KP8NNNC C2: GRM31CR61A107MEA8K L1: B82432T1563K000 D1: 1N4448X-TP"
- note added: "NOTES: - Produce -6V for OLED cell - Circuit based on Fig. 15 in LTC3638 datasheet - Modfified to remove VPRG1 (want only our resistors) - Modified for our voltages"
- note removed: "NOTES: - Produce -6V for OLED cell - Circuit based on Fig. 15 in LTC3638 DS"
Changed lines of the file:
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@@
 	(rectangle
 		(start 17.78 161.29)
-		(end 133.35 194.31)
+		(end 172.72 194.31)
 		(stroke
 			(width 0)
@@
 		)
 	)
-	(text "NOTES:\n- Produce -6V for OLED cell\n- Circuit based on Fig. 15 in LTC3638 DS"
+	(text "NOTES:\n- Produce -6V for OLED cell\n- Circuit based on Fig. 15 in LTC3638\n  datasheet\n- Modfified to remove VPRG1 (want only\n  our resistors)\n- Modified for our voltages"
 		(exclude_from_sim no)
-		(at 21.844 188.976 0)
+		(at 19.558 185.928 0)
 		(effects
 			(font
@@
 		)
 	)
+	(text "C1: CL10B105KP8NNNC\nC2: GRM31CR61A107MEA8K\nL1: B82432T1563K000\nD1: 1N4448X-TP"
+		(exclude_from_sim no)
+		(at 137.668 169.418 0)
+		(effects
+			(font
+				(size 1.27 1.27)
+			)
+			(justify left)
+		)
+	)
 	(junction
 		(at 156.21 77.47)
@@
 	)
 	(junction
-		(at 105.41 184.15)
+		(at 69.85 165.1)
 		(diameter 0)
 		(color 0 0 0 0)
 	)
 	(junction
-		(at 69.85 166.37)
+		(at 105.41 184.15)
 		(diameter 0)
 		(color 0 0 0 0)
 	)
 	(junction
-		(at 74.93 166.37)
+		(at 116.84 173.99)
 		(diameter 0)
 		(color 0 0 0 0)
 	)
 	(junction
-		(at 116.84 173.99)
+		(at 156.21 80.01)
 		(diameter 0)
 		(color 0 0 0 0)
 	)
 	(junction
-		(at 156.21 80.01)
+		(at 74.93 179.07)
 		(diameter 0)
 		(color 0 0 0 0)
@@
 	)
 	(junction
+		(at 74.93 165.1)
+		(diameter 0)
+		(color 0 0 0 0)
+	)
+	(junction
 		(at 260.35 82.55)
 		(diameter 0)
@@
 	)
 	(no_connect
+		(at 76.2 184.15)
+	)
+	(no_connect
 		(at 30.48 86.36)
 	)
@@
 	(wire
 		(pts
+			(xy 74.93 165.1) (xy 74.93 171.45)
+		)
+		(stroke
+			(width 0)
+			(type default)
+		)
+	)
+	(wire
+		(pts
 			(xy 254 102.87) (xy 247.65 102.87)
 		)
@@
 	(wire
 		(pts
+			(xy 74.93 176.53) (xy 76.2 176.53)
+		)
+		(stroke
+			(width 0)
+			(type default)
+		)
+	)
+	(wire
+		(pts
 			(xy 97.79 81.28) (xy 97.79 78.74)
 		)
@@
 	(wire
 		(pts
-			(xy 74.93 166.37) (xy 86.36 166.37)
+			(xy 74.93 165.1) (xy 86.36 165.1)
 		)
 		(stroke
@@
 	(wire
 		(pts
-			(xy 73.66 176.53) (xy 76.2 176.53)
-		)
-		(stroke
-			(width 0)
-			(type default)
-		)
-	)
-	(wire
-		(pts
 			(xy 60.96 68.58) (xy 66.04 68.58)
 		)
@@
 	(wire
 		(pts
-			(xy 74.93 171.45) (xy 74.93 166.37)
+			(xy 255.27 113.03) (xy 247.65 113.03)
 		)
 		(stroke
@@
 	(wire
 		(pts
-			(xy 255.27 113.03) (xy 247.65 113.03)
+			(xy 116.84 181.61) (xy 116.84 193.04)
 		)
 		(stroke
@@
 	(wire
 		(pts
-			(xy 116.84 181.61) (xy 116.84 193.04)
+			(xy 165.1 43.18) (xy 165.1 49.53)
 		)
 		(stroke
@@
 	(wire
 		(pts
-			(xy 165.1 43.18) (xy 165.1 49.53)
+			(xy 60.96 66.04) (xy 66.04 66.04)
 		)
 		(stroke
@@
 	(wire
 		(pts
-			(xy 60.96 66.04) (xy 66.04 66.04)
+			(xy 251.46 140.97) (xy 251.46 138.43)
 		)
 		(stroke
@@
 	(wire
 		(pts
-			(xy 251.46 140.97) (xy 251.46 138.43)
+			(xy 254 128.27) (xy 247.65 128.27)
 		)
 		(stroke
@@
 	(wire
 		(pts
-			(xy 254 128.27) (xy 247.65 128.27)
+			(xy 185.42 152.4) (xy 175.26 152.4)
 		)
 		(stroke
@@
 	(wire
 		(pts
-			(xy 185.42 152.4) (xy 175.26 152.4)
+			(xy 86.36 165.1) (xy 86.36 166.37)
 		)
 		(stroke
@@
 	(wire
 		(pts
+			(xy 74.93 176.53) (xy 74.93 179.07)
+		)
+		(stroke
+			(width 0)
+			(type default)
+		)
+	)
+	(wire
+		(pts
 			(xy 105.41 173.99) (xy 105.41 176.53)
 		)
@@
 	(wire
 		(pts
-			(xy 69.85 166.37) (xy 69.85 168.91)
+			(xy 69.85 165.1) (xy 69.85 168.91)
 		)
 		(stroke
@@
 	(wire
 		(pts
-			(xy 69.85 166.37) (xy 74.93 166.37)
+			(xy 69.85 165.1) (xy 74.93 165.1)
 		)
 		(stroke
@@
 	(wire
 		(pts
-			(xy 73.66 184.15) (xy 73.66 176.53)
-		)
-		(stroke
-			(width 0)
-			(type default)
-		)
-	)
-	(wire
-		(pts
-			(xy 68.58 166.37) (xy 69.85 166.37)
+			(xy 68.58 165.1) (xy 69.85 165.1)
 		)
 		(stroke
@@
 	(wire
 		(pts
-			(xy 76.2 184.15) (xy 73.66 184.15)
-		)
-		(stroke
-			(width 0)
-			(type default)
-		)
-	)
-	(wire
-		(pts
 			(xy 123.19 175.26) (xy 123.19 173.99)
 		)
@@
 		(on_board yes)
 		(dnp no)
-		(property "Reference" "C1"
+		(property "Reference" "C2"
 			(at 114.808 177.8 0)
 			(effects
@@
 			)
 		)
-		(property "Value" "10uF"
+		(property "Value" "100uF"
 			(at 114.808 180.086 0)
 			(effects
@@
 			)
 		)
-		(property "Footprint" "Capacitor_SMD:C_1210_3225Metric"
+		(property "Footprint" "Capacitor_SMD:C_1206_3216Metric"
 			(at 116.84 179.07 0)
 			(effects
@@
 			(project "e90-dsi-split"
 				(path "/06866490-d885-4e24-8e91-5348d6179fe2"
-					(reference "C1")
+					(reference "C2")
 					(unit 1)
 				)
@@
 		(on_board yes)
 		(dnp no)
-		(property "Reference" "C2"
+		(property "Reference" "C1"
 			(at 65.532 169.926 0)
 			(effects
@@
 			(project ""
 				(path "/06866490-d885-4e24-8e91-5348d6179fe2"
-					(reference "C2")
+					(reference "C1")
 					(unit 1)
 				)
@@
 			)
 		)
-		(property "Value" "220uH"
+		(property "Value" "56uH"
 			(at 100.33 171.45 90)
 			(effects
@@
 			)
 		)
-		(property "Footprint" "Inductor_SMD:L_TDK_NLV32_3.2x2.5mm"
+		(property "Footprint" "Inductor_SMD:L_1812_4532Metric"
 			(at 100.33 173.99 0)
 			(effects
@@
 	(symbol
 		(lib_id "power:+5V")
-		(at 68.58 166.37 90)
+		(at 68.58 165.1 90)
 		(unit 1)
 		(exclude_from_sim no)
@@
 		(fields_autoplaced yes)
 		(property "Reference" "#PWR023"
-			(at 72.39 166.37 0)
+			(at 72.39 165.1 0)
 			(effects
 				(font
@@
 		)
 		(property "Value" "LCD0_BL+"
-			(at 64.77 166.3699 90)
+			(at 64.77 165.0999 90)
 			(effects
 				(font
@@
 		)
 		(property "Footprint" ""
-			(at 68.58 166.37 0)
+			(at 68.58 165.1 0)
 			(effects
 				(font
@@
 		)
 		(property "Datasheet" ""
-			(at 68.58 166.37 0)
+			(at 68.58 165.1 0)
 			(effects
 				(font
@@
 		)
 		(property "Description" "Power symbol creates a global label with name \"+5V\""
-			(at 68.58 166.37 0)
+			(at 68.58 165.1 0)
 			(effects
 				(font
@@
 			)
 		)
-		(property "Footprint" "Diode_SMD:D_SOD-123"
+		(property "Footprint" "Diode_SMD:D_SOD-523"
 			(at 99.06 187.96 90)
 			(effects

Commit message: updates post rework
Parts:
- R1: value 65k -> 130k
- R2: value 10k -> 20k
Connections:
- net at R1.2, R2.1, U3.9 (VFB): no longer D1.1 (K)
- net at L1.1, U3.1 (SW): now also D1.1 (K)
Other:
- moved on the sheet: D1, L1
Changed lines of the file:
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@@
 	)
 	(junction
-		(at 99.06 193.04)
-		(diameter 0)
-		(color 0 0 0 0)
-	)
-	(junction
 		(at 74.93 165.1)
 		(diameter 0)
@@
 	)
 	(junction
-		(at 99.06 184.15)
+		(at 260.35 77.47)
 		(diameter 0)
 		(color 0 0 0 0)
 	)
 	(junction
-		(at 260.35 77.47)
+		(at 105.41 173.99)
 		(diameter 0)
 		(color 0 0 0 0)
 	)
 	(junction
-		(at 105.41 173.99)
+		(at 97.79 193.04)
 		(diameter 0)
 		(color 0 0 0 0)
@@
 	)
 	(junction
+		(at 97.79 173.99)
+		(diameter 0)
+		(color 0 0 0 0)
+	)
+	(junction
 		(at 260.35 64.77)
 		(diameter 0)
@@
 	(wire
 		(pts
+			(xy 97.79 193.04) (xy 105.41 193.04)
+		)
+		(stroke
+			(width 0)
+			(type default)
+		)
+	)
+	(wire
+		(pts
 			(xy 185.42 144.78) (xy 185.42 152.4)
 		)
@@
 	(wire
 		(pts
-			(xy 254 100.33) (xy 247.65 100.33)
+			(xy 97.79 173.99) (xy 99.06 173.99)
 		)
 		(stroke
@@
 	(wire
 		(pts
-			(xy 30.48 55.88) (xy 35.56 55.88)
+			(xy 254 100.33) (xy 247.65 100.33)
 		)
 		(stroke
@@
 	(wire
 		(pts
-			(xy 60.96 81.28) (xy 68.58 81.28)
+			(xy 30.48 55.88) (xy 35.56 55.88)
 		)
 		(stroke
@@
 	(wire
 		(pts
-			(xy 149.86 77.47) (xy 156.21 77.47)
+			(xy 60.96 81.28) (xy 68.58 81.28)
 		)
 		(stroke
@@
 	(wire
 		(pts
-			(xy 76.2 173.99) (xy 72.39 173.99)
+			(xy 149.86 77.47) (xy 156.21 77.47)
 		)
 		(stroke
@@
 	(wire
 		(pts
-			(xy 260.35 83.82) (xy 260.35 82.55)
+			(xy 76.2 173.99) (xy 72.39 173.99)
 		)
 		(stroke
@@
 	(wire
 		(pts
-			(xy 260.35 64.77) (xy 260.35 67.31)
+			(xy 260.35 83.82) (xy 260.35 82.55)
 		)
 		(stroke
@@
 	(wire
 		(pts
-			(xy 184.15 142.24) (xy 195.58 142.24)
+			(xy 260.35 64.77) (xy 260.35 67.31)
 		)
 		(stroke
@@
 	(wire
 		(pts
-			(xy 96.52 184.15) (xy 99.06 184.15)
+			(xy 184.15 142.24) (xy 195.58 142.24)
 		)
 		(stroke
@@
 	(wire
 		(pts
-			(xy 102.87 173.99) (xy 105.41 173.99)
+			(xy 104.14 173.99) (xy 105.41 173.99)
 		)
 		(stroke
@@
 	(wire
 		(pts
-			(xy 99.06 190.5) (xy 99.06 193.04)
+			(xy 97.79 181.61) (xy 97.79 193.04)
 		)
 		(stroke
@@
 	(wire
 		(pts
-			(xy 86.36 193.04) (xy 99.06 193.04)
+			(xy 86.36 193.04) (xy 97.79 193.04)
 		)
 		(stroke
@@
 	(wire
 		(pts
-			(xy 99.06 184.15) (xy 105.41 184.15)
+			(xy 96.52 184.15) (xy 105.41 184.15)
 		)
 		(stroke
@@
 	(wire
 		(pts
-			(xy 90.17 76.2) (xy 97.79 76.2)
+			(xy 97.79 173.99) (xy 97.79 176.53)
 		)
 		(stroke
@@
 	(wire
 		(pts
-			(xy 31.75 144.78) (xy 25.4 144.78)
+			(xy 90.17 76.2) (xy 97.79 76.2)
 		)
 		(stroke
@@
 	(wire
 		(pts
-			(xy 105.41 193.04) (xy 99.06 193.04)
+			(xy 31.75 144.78) (xy 25.4 144.78)
 		)
 		(stroke
@@
 	(wire
 		(pts
-			(xy 99.06 184.15) (xy 99.06 185.42)
-		)
-		(stroke
-			(width 0)
-			(type default)
-		)
-	)
-	(wire
-		(pts
 			(xy 254 125.73) (xy 247.65 125.73)
 		)
@@
 			)
 		)
-		(property "Value" "10k"
+		(property "Value" "20k"
 			(at 106.934 188.976 0)
 			(effects
@@
 	(symbol
 		(lib_id "Device:L_Small")
-		(at 100.33 173.99 90)
+		(at 101.6 173.99 90)
 		(unit 1)
 		(exclude_from_sim no)
@@
 		(fields_autoplaced yes)
 		(property "Reference" "L1"
-			(at 100.33 168.91 90)
+			(at 101.6 168.91 90)
 			(effects
 				(font
@@
 		)
 		(property "Value" "56uH"
-			(at 100.33 171.45 90)
+			(at 101.6 171.45 90)
 			(effects
 				(font
@@
 		)
 		(property "Footprint" "Inductor_SMD:L_1812_4532Metric"
-			(at 100.33 173.99 0)
+			(at 101.6 173.99 0)
 			(effects
 				(font
@@
 		)
 		(property "Datasheet" "~"
-			(at 100.33 173.99 0)
+			(at 101.6 173.99 0)
 			(effects
 				(font
@@
 		)
 		(property "Description" "Inductor, small symbol"
-			(at 100.33 173.99 0)
+			(at 101.6 173.99 0)
 			(effects
 				(font
@@
 	(symbol
 		(lib_id "Device:D_Zener_Small")
-		(at 99.06 187.96 270)
+		(at 97.79 179.07 270)
 		(unit 1)
 		(exclude_from_sim no)
@@
 		(dnp no)
 		(property "Reference" "D1"
-			(at 100.584 187.96 90)
+			(at 96.774 179.07 90)
 			(effects
 				(font
 					(size 1.27 1.27)
 				)
-				(justify left)
+				(justify right)
 			)
 		)
 		(property "Value" "~"
-			(at 101.6 189.23 90)
+			(at 100.33 180.34 90)
 			(effects
 				(font
@@
 		)
 		(property "Footprint" "Diode_SMD:D_SOD-523"
-			(at 99.06 187.96 90)
+			(at 97.79 179.07 90)
 			(effects
 				(font
@@
 		)
 		(property "Datasheet" "~"
-			(at 99.06 187.96 90)
+			(at 97.79 179.07 90)
 			(effects
 				(font
@@
 		)
 		(property "Description" "Zener diode, small symbol"
-			(at 99.06 187.96 0)
+			(at 97.79 179.07 0)
 			(effects
 				(font
@@
 			)
 		)
-		(property "Value" "65k"
+		(property "Value" "130k"
 			(at 103.886 180.34 0)
 			(effects
