File: v0/e90-dsi-split.kicad_sch (KiCad schematic)
At the start: 21 parts, among them J1 3-2328724-1, J2 BM23PF0.8-40DP-0.35V_51_, U1 ICM-42605, U3 LTC3638xMSE

Commit message: v2: start v2
Parts:
- removed D1: ~, Diode_SMD:D_SOD-523, symbol Device:D_Zener_Small
- removed TP3: MVDD Test, TestPoint:TestPoint_Pad_1.0x1.0mm, symbol Connector:TestPoint
- removed TP4: VREF1 Test, TestPoint:TestPoint_Pad_1.0x1.0mm, symbol Connector:TestPoint
- removed TP5: ELVDD Test, TestPoint:TestPoint_Pad_1.0x1.0mm, symbol Connector:TestPoint
- removed TP7: VGSP Test, TestPoint:TestPoint_Pad_1.0x1.0mm, symbol Connector:TestPoint
- removed TP8: VGMP Test, TestPoint:TestPoint_Pad_1.0x1.0mm, symbol Connector:TestPoint
- added C10, C11, C12, C13, C3, C4, C5, C6, C7, C8, C9: C_Small, symbol Device:C_Small
- added D2, D3: D_Schottky_Small, symbol Device:D_Schottky_Small
- TP11: value -5V5 Screen -> -6V Src
- TP2: value -5V5 Screen -> -6V Screen
Connections:
- net -6V: now also D3.2 (A)
- net AVEE: now also C13.1
- net ELVDD: now also C4.2
- net GND: now also C1.2, C2.1, L1.2, R1.1, C10.1, C11.2, C12.1, C13.2, C3.2, C4.1, C5.2, C6.2, C7.2, C8.2, C9.2, D2.1 (K); no longer J2.36, J2.38
- net LCD0_BL+: no longer C1.1, J1.29, J1.30, J1.31, U3.14 (RUN), U3.3 (VIN)
- net OCP_VDD2: now also C10.2
- net VCOM: now also C3.1, D2.2 (A)
- net VDD1V8_SYS: now also C12.2; no longer J2.MP2, J2.MP4
- net VDD3V3_SYS: now also C1.1, U3.14 (RUN), U3.3 (VIN)
- net VGMP: now also C7.1
- net VGSP: now also C6.1
- net VREF1: now also C5.1
- net VREF2: now also C9.1
- net VREF3: now also C8.1
- net at L1.1, U3.1 (SW): now also D3.1 (K)
- removed net LCD0_BL-: C1.2, C2.1, J1.24, J1.25, J1.26, J1.27, L1.2, R1.1
- new net EN_EXT_VDD: J2.36
- new net VDD: C11.1, J2.MP2, J2.MP4
- no-connect marks 21 -> 26
Other:
- moved on the sheet: J2, TP1, TP10, TP11, TP2, TP9

Commit message: v2: continue
Parts:
- added U2: LicheeRV_Nano, Module:LicheeRV_Nano, symbol Core_moudle:LicheeRV_Nano
- C10, C11, C12, C13, C3, C4, C5, C6, C7, C8, C9: footprint (none) -> Capacitor_SMD:C_0603_1608Metric
- D2, D3: footprint (none) -> Diode_SMD:D_SOD-123
- L1: value 56uH -> 51uH
Connections:
- net LCD0_BL+ is gone; now on net VDD3V3_SYS: TP10.1
- net VDD3V3_SYS: no longer C1.1, FPC1.2, U1.5 (VDDIO), U1.8 (VDD), U3.14 (RUN), U3.3 (VIN)
- new net +5V: C1.1, U2.13 (VSYS), U3.14 (RUN), U3.3 (VIN)
- new net VDD3V3_I2C: FPC1.2, U1.5 (VDDIO), U1.8 (VDD)
Other:
- note added: "Pin Interface"
- moved on the sheet: C10, C11, C12, C13, C3, C4, C5, C6, C7, C8, C9, D2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

Commit message: v2: more updates
Parts:
- added C14: C_Small, Capacitor_SMD:C_0603_1608Metric, symbol Device:C_Small
Connections:
- net IM_0 is gone; now on net GND: J2.27
- net GND: now also J2.38, C14.1
- net MVDD: now also C14.2
- net VDD3V3_SYS: no longer TP10.1
- net LCD0_BL+: now reaches J1.29
- net LCD0_BL+: now also J1.30, J1.31, TP10.1
- no-connect marks 26 -> 23
Changed lines of the file:
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@@
 	)
 	(junction
+		(at 257.81 67.31)
+		(diameter 0)
+		(color 0 0 0 0)
+	)
+	(junction
 		(at 116.84 193.04)
 		(diameter 0)
@@
 	)
 	(junction
+		(at 19.05 63.5)
+		(diameter 0)
+		(color 0 0 0 0)
+	)
+	(junction
+		(at 19.05 68.58)
+		(diameter 0)
+		(color 0 0 0 0)
+	)
+	(junction
 		(at 81.28 90.17)
 		(diameter 0)
@@
 	)
 	(no_connect
-		(at 252.73 64.77)
-	)
-	(no_connect
 		(at 69.85 71.12)
 	)
@@
 	)
 	(no_connect
-		(at 252.73 67.31)
-	)
-	(no_connect
 		(at 257.81 72.39)
 	)
@@
 	)
 	(no_connect
-		(at 252.73 69.85)
-	)
-	(no_connect
 		(at 252.73 74.93)
 	)
@@
 	(wire
 		(pts
-			(xy 19.05 53.34) (xy 19.05 78.74)
+			(xy 19.05 53.34) (xy 19.05 63.5)
 		)
 		(stroke
@@
 	(wire
 		(pts
-			(xy 34.29 63.5) (xy 39.37 63.5)
+			(xy 189.23 36.83) (xy 189.23 39.37)
 		)
 		(stroke
@@
 	(wire
 		(pts
-			(xy 189.23 36.83) (xy 189.23 39.37)
+			(xy 194.31 142.24) (xy 200.66 142.24)
 		)
 		(stroke
@@
 	(wire
 		(pts
-			(xy 194.31 142.24) (xy 200.66 142.24)
+			(xy 254 85.09) (xy 254 87.63)
 		)
 		(stroke
@@
 	(wire
 		(pts
-			(xy 254 85.09) (xy 254 87.63)
+			(xy 64.77 81.28) (xy 69.85 81.28)
+		)
+		(stroke
+			(width 0)
+			(type default)
+		)
+	)
+	(wire
+		(pts
+			(xy 257.81 67.31) (xy 269.24 67.31)
 		)
 		(stroke
@@
 	(wire
 		(pts
+			(xy 33.02 63.5) (xy 39.37 63.5)
+		)
+		(stroke
+			(width 0)
+			(type default)
+		)
+	)
+	(wire
+		(pts
 			(xy 31.75 86.36) (xy 31.75 83.82)
 		)
@@
 	(wire
 		(pts
+			(xy 19.05 63.5) (xy 27.94 63.5)
+		)
+		(stroke
+			(width 0)
+			(type default)
+		)
+	)
+	(wire
+		(pts
 			(xy 64.77 50.8) (xy 69.85 50.8)
 		)
@@
 	(wire
 		(pts
+			(xy 19.05 68.58) (xy 39.37 68.58)
+		)
+		(stroke
+			(width 0)
+			(type default)
+		)
+	)
+	(wire
+		(pts
 			(xy 24.13 86.36) (xy 31.75 86.36)
 		)
@@
 	(wire
 		(pts
-			(xy 34.29 68.58) (xy 39.37 68.58)
+			(xy 34.29 81.28) (xy 39.37 81.28)
 		)
 		(stroke
@@
 	(wire
 		(pts
-			(xy 34.29 81.28) (xy 39.37 81.28)
+			(xy 69.85 173.99) (xy 69.85 175.26)
 		)
 		(stroke
@@
 	(wire
 		(pts
-			(xy 69.85 173.99) (xy 69.85 175.26)
+			(xy 34.29 71.12) (xy 39.37 71.12)
 		)
 		(stroke
@@
 	(wire
 		(pts
-			(xy 34.29 71.12) (xy 39.37 71.12)
+			(xy 64.77 38.1) (xy 81.28 38.1)
 		)
 		(stroke
@@
 	(wire
 		(pts
-			(xy 64.77 38.1) (xy 81.28 38.1)
+			(xy 257.81 67.31) (xy 257.81 64.77)
 		)
 		(stroke
@@
 	(wire
 		(pts
-			(xy 27.94 68.58) (xy 27.94 76.2)
+			(xy 27.94 69.85) (xy 27.94 76.2)
 		)
 		(stroke
@@
 	(wire
 		(pts
+			(xy 19.05 63.5) (xy 19.05 68.58)
+		)
+		(stroke
+			(width 0)
+			(type default)
+		)
+	)
+	(wire
+		(pts
 			(xy 69.85 165.1) (xy 69.85 168.91)
 		)
@@
 	(wire
 		(pts
+			(xy 257.81 69.85) (xy 257.81 67.31)
+		)
+		(stroke
+			(width 0)
+			(type default)
+		)
+	)
+	(wire
+		(pts
 			(xy 259.08 110.49) (xy 252.73 110.49)
 		)
@@
 	(wire
 		(pts
+			(xy 257.81 64.77) (xy 252.73 64.77)
+		)
+		(stroke
+			(width 0)
+			(type default)
+		)
+	)
+	(wire
+		(pts
 			(xy 74.93 179.07) (xy 74.93 193.04)
 		)
@@
 	(wire
 		(pts
+			(xy 252.73 69.85) (xy 257.81 69.85)
+		)
+		(stroke
+			(width 0)
+			(type default)
+		)
+	)
+	(wire
+		(pts
+			(xy 19.05 68.58) (xy 19.05 78.74)
+		)
+		(stroke
+			(width 0)
+			(type default)
+		)
+	)
+	(wire
+		(pts
 			(xy 96.52 184.15) (xy 105.41 184.15)
 		)
@@
 	(wire
 		(pts
+			(xy 252.73 67.31) (xy 257.81 67.31)
+		)
+		(stroke
+			(width 0)
+			(type default)
+		)
+	)
+	(wire
+		(pts
 			(xy 72.39 35.56) (xy 73.66 35.56)
 		)
@@
 		)
 	)
+	(label "LCD0_BL+"
+		(at 269.24 67.31 180)
+		(effects
+			(font
+				(size 1.27 1.27)
+			)
+			(justify right bottom)
+		)
+	)
 	(label "OCP_OUT"
 		(at 69.85 73.66 180)
@@
 	)
 	(label "VCOM"
-		(at 27.94 68.58 270)
+		(at 27.94 69.85 270)
 		(effects
 			(font
@@
 			)
 		)
-		(property "Value" "VDD3V3_SYS"
-			(at 146.05 30.48 0)
+		(property "Value" "LCD0_BL+"
+			(at 148.59 34.2899 0)
 			(effects
 				(font
 					(size 1.27 1.27)
 				)
+				(justify left)
 			)
 		)
@@
 					(unit 1)
 				)
+			)
+		)
+	)
+	(symbol
+		(lib_id "Device:C_Small")
+		(at 30.48 63.5 90)
+		(unit 1)
+		(exclude_from_sim no)
+		(in_bom yes)
+		(on_board yes)
+		(dnp no)
+		(fields_autoplaced yes)
+		(property "Reference" "C14"
+			(at 30.4863 57.15 90)
+			(effects
+				(font
+					(size 1.27 1.27)
+				)
+			)
+		)
+		(property "Value" "C_Small"
+			(at 30.4863 59.69 90)
+			(effects
+				(font
+					(size 1.27 1.27)
+				)
+			)
+		)
+		(property "Footprint" "Capacitor_SMD:C_0603_1608Metric"
+			(at 30.48 63.5 0)
+			(effects
+				(font
+					(size 1.27 1.27)
+				)
+				(hide yes)
+			)
+		)
+		(property "Datasheet" "~"
+			(at 30.48 63.5 0)
+			(effects
+				(font
+					(size 1.27 1.27)
+				)
+				(hide yes)
+			)
+		)
+		(property "Description" "Unpolarized capacitor, small symbol"
+			(at 30.48 63.5 0)
+			(effects
+				(font
+					(size 1.27 1.27)
+				)
+				(hide yes)
+			)
+		)
+		(pin "2"
+		)
+		(pin "1"
+		)
+		(instances
+			(project "e90-dsi-split"
+				(path "/06866490-d885-4e24-8e91-5348d6179fe2"
+					(reference "C14")
+					(unit 1)
+				)
